File: sweatyHands_sch.kicad_sch (KiCad schematic)
At the start: 96 parts, among them J1 USB_C_Receptacle_USB2.0_16P, J2 Barrel_Jack, J3 Conn_02x06_Odd_Even, J4 105-1103-001, J5 105-1103-001, J6 Conn_01x04_Socket, Q1 UMH3N, Q2 MMBTA06, Q3 MMBTA06, Q4 AON6266E, Q5 FDC5614P, Q6 AON6266E, Q7 FDC5614P, Q8 AON6266E, Q9 AON6266E, SW1 SW_SPST, U1 TLV1117LV-3.3, U2 TPS2553DBVR, U3 USBLC6-2SC6, U4 TPS2116DRL, U5 ESP32-WROOM-32E, U6 CP2104, U7 LMR14020SDDAR

Commit message: First Complete Draft done
Parts:
- removed Q5, Q7: FDC5614P, Extra:TSOT23-6_419BL_ONS, symbol Simulation_SPICE:PMOS
- removed Q8, Q9: AON6266E, Extra:AON6482, symbol Simulation_SPICE:NMOS
- added MOSFET1, MOSFET2: FDC5614P, TSOT23-6_419BL_ONS, symbol FDC5614P:FDC5614P
- added Q5, Q7: T2N7002BK_LM, Extra:SOT23_TOS-M, symbol Simulation_SPICE:NMOS
- Q4, Q6: value AON6266E -> T2N7002BK_LM; footprint Extra:AON6482 -> Extra:SOT23_TOS-M
- renumbered C21 to C15, C15 to C16, C16 to C17, C17 to C18, C18 to C19, C19 to C20, C20 to C21, Q2 to Q1, Q3 to Q2, Q1 to Q3, R17 to R15, R15 to R16, R16 to R17, R19 to R18, R33 to R19, R18 to R20, R20 to R21, R21 to R24, R24 to R25, R25 to R26, R26 to R27, R27 to R28, R28 to R29, R29 to R30, R30 to R31, R31 to R32, R32 to R33
Connections:
- net GPIO34 is gone; now on net GPIO25: J3.7 (Pin_7)
- net +36V: now also MOSFET1.4, MOSFET2.4
- net Digi_GND: now also Q5.3 (S), Q7.3 (S)
- net GND: now also J3.10 (Pin_10); no longer J3.9 (Pin_9)
- net GPIO18: now also J3.8 (Pin_8); no longer J3.4 (Pin_4)
- net GPIO19: now also J3.6 (Pin_6)
- net GPIO25: no longer J3.6 (Pin_6)
- net GPIO26: now also J3.9 (Pin_9); no longer J3.8 (Pin_8)
- net GPIO27: now also J3.4 (Pin_4); no longer J3.10 (Pin_10)
- net LEFT_HAND: now also MOSFET1.1, MOSFET1.2, MOSFET1.5, MOSFET1.6, Q5.1 (D); no longer Q6.1 (D)
- net RIGHT_HAND: now also Q6.1 (D), MOSFET2.1, MOSFET2.2, MOSFET2.5, MOSFET2.6
- net at D4.2 (A), R22.2, R23.1: now also MOSFET1.3
- net at R30.1: now also Q6.2 (G)
- net at R26.2: now also Q5.2 (G); no longer Q6.2 (G)
- net at R32.2: now also Q7.1 (D)
- net at R34.1: now also Q7.2 (G)
- net at D5.2 (A), R31.2, R32.1: now also MOSFET2.3
Other:
- moved on the sheet: C15, D4, D5, J4, J5, Q1, Q2, R15, R18, R19, R20, R21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

Commit message: meow
Parts:
- added Pot1: 1, Resistor_THT:R_Axial_DIN0204_L3.6mm_D1.6mm_P2.54mm_Vertical, symbol Device:R
- added R38: 5000, Resistor_SMD:R_0603_1608Metric_Pad0.98x0.95mm_HandSolder, symbol Device:R
Connections:
- net +3.3V: now also R38.1
- net GND: now also Pot1.2
- net at U5.26 (IO4): now also Pot1.1, R38.2

Commit message: Update
Parts:
- removed Pot1: 1, Resistor_THT:R_Axial_DIN0204_L3.6mm_D1.6mm_P2.54mm_Vertical, symbol Device:R
- added J7: PDB181-K420K-502B, CONN3_PDB181-K420K-502B_BRN, symbol PDB181-K420K-502B:PDB181-K420K-502B
- added R39: PTV09A-4015U-A204, POT_PTV09A-4x15x-xxxx_BRN, symbol 2025-09-19_05-32-43:PTV09A-4015U-A204
- added R40: 0R, Resistor_SMD:R_0603_1608Metric_Pad0.98x0.95mm_HandSolder, symbol Device:R_Small
Connections:
- net GND: now also R39.2
- net RIGHT_HAND: now also J7.2, R40.1; no longer MOSFET2.1, MOSFET2.2, MOSFET2.5, MOSFET2.6, Q6.1 (D)
- net at R38.2, U5.26 (IO4): now also R39.1
- new net: J7.1, MOSFET2.1, MOSFET2.2, MOSFET2.5, MOSFET2.6, Q6.1 (D), R40.2
