File: sweatyHands_sch.kicad_pcb (KiCad board)
At the start: 4 copper layers, 100 x 100 mm, 90 parts, among them J2 Conn_01x04_Socket, J3 Conn_02x06_Odd_Even, J4 Barrel_Jack, J5 USB_C_Receptacle_USB2.0_16P, J7 Conn_01x02_Socket, Q1 UMH3N, Q10 2N3904, Q3 AO3400A, Q4 DMG2305UX-13, Q5 DMG2305UX-13, Q6 AO3400A, Q7 MMBT3904, Q8 MMBT3904, Q9 2N3904, SW1 SW_SPST, U1 ESP32-WROOM-32E, U2 TPS54202DDCT, U4 TLV1117LV-3.3, U5 TPS2116DRL, U6 TPS2553DBVR, U7 CP2104, U8 USBLC6-2SC6

Commit message: ABout halfway done with PCB
Parts:
- removed C22, C23: 22u, Capacitor_SMD:C_0805_2012Metric_Pad1.18x1.45mm_HandSolder
- removed C24: 75p, Capacitor_SMD:C_0805_2012Metric_Pad1.18x1.45mm_HandSolder
- removed CR2: MMSZ5236B-7-F, Extra:SOD123_DIO
- removed F3: Polyfuse 1.2-1.5A hold, Fuse:Fuse_0805_2012Metric_Pad1.15x1.40mm_HandSolder
- removed J7: Conn_01x02_Socket, Connector:Banana_Jack_2Pin
- removed Q10: 2N3904, Package_TO_SOT_THT:TO-92_Inline
- removed the R15 at (254.5, 92.0)
- removed the R16 at (254.5, 95.0)
- removed R38: 47K, Resistor_SMD:R_0805_2012Metric
- removed R39: 240K, Resistor_SMD:R_0805_2012Metric
- removed R40: 100K, Resistor_SMD:R_0805_2012Metric
- removed the R6 at (250.1, 92.0)
- removed the U5 at (146.6, 91.3)
- removed the U6 at (126.3, 66.7)
- added C1: 22u, Capacitor_SMD:C_0603_1608Metric_Pad1.08x0.95mm_HandSolder, F.Cu at (166.0, 84.4)
- added C2: 22u, Capacitor_SMD:C_0603_1608Metric_Pad1.08x0.95mm_HandSolder, F.Cu at (157.7, 84.2)
- added C3: 0.1u, Capacitor_SMD:C_0603_1608Metric_Pad1.08x0.95mm_HandSolder, F.Cu at (189.1, 73.0)
- added C4: 100n, Capacitor_SMD:C_0603_1608Metric_Pad1.08x0.95mm_HandSolder, F.Cu at (219.1, 85.0)
- added C5: 1u, Capacitor_SMD:C_0603_1608Metric_Pad1.08x0.95mm_HandSolder, F.Cu at (179.2, 80.8)
- added C6: 1u, Capacitor_SMD:C_0603_1608Metric_Pad1.08x0.95mm_HandSolder, F.Cu at (177.0, 88.8)
- added D5: TFZVTR10B, Extra:DIO_TDZVT_ROM-M, F.Cu at (224.2, 112.3)
- added F1: Polyfuse 500ma, Fuse:Fuse_0805_2012Metric_Pad1.15x1.40mm_HandSolder, F.Cu at (186.9, 67.2)
- added J5: 105-1103-001, Extra:CONN_105-1102-001, F.Cu at (156.1, 141.5)
- added J6: Conn_01x04_Socket, Connector_PinHeader_2.54mm:PinHeader_1x04_P2.54mm_Vertical, F.Cu at (219.0, 97.8)
- added Q2: MMBTA06, Extra:TRANS_MMBTA06, F.Cu at (257.0, 76.7)
- added R1: 1K, Resistor_SMD:R_0603_1608Metric_Pad0.98x0.95mm_HandSolder, F.Cu at (132.9, 79.0)
- added R17: 22K, Resistor_SMD:R_0603_1608Metric_Pad0.98x0.95mm_HandSolder, F.Cu at (235.4, 92.5)
- added R18: 10K, Resistor_SMD:R_0603_1608Metric_Pad0.98x0.95mm_HandSolder, F.Cu at (235.4, 94.2)
- added R19: 24, Resistor_SMD:R_0603_1608Metric_Pad0.98x0.95mm_HandSolder, F.Cu at (235.4, 96.0)
- added R2: 1K, Resistor_SMD:R_0603_1608Metric_Pad0.98x0.95mm_HandSolder, F.Cu at (132.9, 73.4)
- added R20: 100R, Resistor_SMD:R_0603_1608Metric_Pad0.98x0.95mm_HandSolder, F.Cu at (235.4, 97.7)
- added R3: 1K, Resistor_SMD:R_0603_1608Metric_Pad0.98x0.95mm_HandSolder, F.Cu at (132.6, 85.2)
- added R4: 1K, Resistor_SMD:R_0603_1608Metric_Pad0.98x0.95mm_HandSolder, F.Cu at (232.6, 92.5)
- added U1: TLV1117LV-3.3, Package_SON:WSON-8-1EP_4x4mm_P0.8mm_EP2.2x3mm, F.Cu at (161.7, 86.7)
- added U7: LMR14020SDDAR, Extra:DDA0008E_N, F.Cu at (186.1, 112.0)
- C10, C8: value 22u -> 100n; footprint Capacitor_SMD:C_0805_2012Metric_Pad1.18x1.45mm_HandSolder -> Capacitor_SMD:C_0603_1608Metric_Pad1.08x0.95mm_HandSolder
- C11: value 22u -> 4u7
- C12: value 100n -> 4u7; footprint Capacitor_SMD:C_0805_2012Metric_Pad1.18x1.45mm_HandSolder -> Capacitor_SMD:C_0603_1608Metric_Pad1.08x0.95mm_HandSolder
- C13, C14, C7: footprint Capacitor_SMD:C_0805_2012Metric_Pad1.18x1.45mm_HandSolder -> Capacitor_SMD:C_0603_1608Metric_Pad1.08x0.95mm_HandSolder
- C15: value 100n -> 10u; footprint Capacitor_SMD:C_0805_2012Metric_Pad1.18x1.45mm_HandSolder -> Capacitor_SMD:C_0603_1608Metric_Pad1.08x0.95mm_HandSolder
- C16: value 4u7 -> 22n; footprint Capacitor_SMD:C_0805_2012Metric_Pad1.18x1.45mm_HandSolder -> Capacitor_SMD:C_0603_1608Metric_Pad1.08x0.95mm_HandSolder
- C17: value 4u7 -> 0.1u; footprint Capacitor_SMD:C_0805_2012Metric_Pad1.18x1.45mm_HandSolder -> Resistor_SMD:R_0603_1608Metric_Pad0.98x0.95mm_HandSolder
- C19, C9: value 100n -> 22u; footprint Capacitor_SMD:C_0805_2012Metric_Pad1.18x1.45mm_HandSolder -> Capacitor_SMD:C_0603_1608Metric_Pad1.08x0.95mm_HandSolder
- C20: value 10u -> 22u; footprint Capacitor_SMD:C_0805_2012Metric_Pad1.18x1.45mm_HandSolder -> Capacitor_SMD:C_0603_1608Metric_Pad1.08x0.95mm_HandSolder
- C21: value 0.1u -> 100n; footprint Capacitor_SMD:C_0805_2012Metric_Pad1.18x1.45mm_HandSolder -> Capacitor_SMD:C_0603_1608Metric_Pad1.08x0.95mm_HandSolder
- CR1: value MMSZ5236B-7-F -> SMF36CA; footprint Extra:SOD123_DIO -> Extra:SOD-123F_LTF
- D1: value LED_RGBA -> PESD5V0S1UL_315; footprint LED_SMD:LED_RGB_Wuerth-PLCC4_3.2x2.8mm_150141M173100 -> Extra:DIO_PESD5V0S1UL_315
- D3: value PESD5V0S1UL_315 -> LED_RGBA; footprint Extra:DIO_PESD5V0S1UL_315 -> LED_SMD:LED_RGB_Wuerth-PLCC4_3.2x2.8mm_150141M173100
- D4: value SS34 -> TFZVTR10B; footprint Diode_SMD:D_SMA -> Extra:DIO_TDZVT_ROM-M
- F2: value Polyfuse 500ma -> Polyfuse 1.2-1.5A hold
- J2: value Conn_01x04_Socket -> Barrel_Jack; footprint Connector_PinHeader_2.54mm:PinHeader_1x04_P2.54mm_Vertical -> Extra:CUI_PJ-002B
- J4: value Barrel_Jack -> 105-1103-001; footprint Extra:CUI_PJ-002B -> Extra:CONN_105-1102-001
- L1: value 15u -> MPZ2012S221AT000; footprint Inductor_SMD:L_0805_2012Metric -> Extra:IND_2012_TDK
- L3: value MPZ2012S221AT000 -> 5.5u; footprint Extra:IND_2012_TDK -> Inductor_SMD:L_0805_2012Metric
- Q3: value AO3400A -> MMBTA06; footprint Package_TO_SOT_SMD:SOT-23 -> Extra:TRANS_MMBTA06
- Q4: value DMG2305UX-13 -> AON6266E; footprint Extra:SOT91P240X110-3N -> Extra:AON6482
- Q5: value DMG2305UX-13 -> FDC5614P; footprint Extra:SOT91P240X110-3N -> Extra:TSOT23-6_419BL_ONS
- Q6: value AO3400A -> AON6266E; footprint Package_TO_SOT_SMD:SOT-23 -> Extra:AON6482
- Q7: value MMBT3904 -> FDC5614P; footprint Package_TO_SOT_SMD:SOT-23 -> Extra:TSOT23-6_419BL_ONS
- Q8: value MMBT3904 -> AON6266E; footprint Package_TO_SOT_SMD:SOT-23 -> Extra:AON6482
- Q9: value 2N3904 -> AON6266E; footprint Package_TO_SOT_THT:TO-92_Inline -> Extra:AON6482
- R10: value 1K -> 240K; footprint Resistor_SMD:R_0805_2012Metric -> Resistor_SMD:R_0603_1608Metric_Pad0.98x0.95mm_HandSolder
- R11: value 4K7 -> 100K; footprint Resistor_SMD:R_0805_2012Metric -> Resistor_SMD:R_0603_1608Metric_Pad0.98x0.95mm_HandSolder
- R12: value 4K7 -> 10K; footprint Resistor_SMD:R_0805_2012Metric -> Resistor_SMD:R_0603_1608Metric_Pad0.98x0.95mm_HandSolder
- R13: value 100K -> 10K; footprint Resistor_SMD:R_0805_2012Metric -> Resistor_SMD:R_0603_1608Metric_Pad0.98x0.95mm_HandSolder
- R14: footprint Resistor_SMD:R_0805_2012Metric -> Resistor_SMD:R_0201_0603Metric_Pad0.64x0.40mm_HandSolder
- R15: renamed from R17; footprint Resistor_SMD:R_0805_2012Metric -> Resistor_SMD:R_0603_1608Metric_Pad0.98x0.95mm_HandSolder
- R16: renamed from R18; footprint Resistor_SMD:R_0805_2012Metric -> Resistor_SMD:R_0603_1608Metric_Pad0.98x0.95mm_HandSolder
- R21: value 49.9R -> 10K; footprint Resistor_SMD:R_0805_2012Metric -> Resistor_SMD:R_0603_1608Metric_Pad0.98x0.95mm_HandSolder
- R22, R26: footprint Resistor_SMD:R_0805_2012Metric -> Resistor_SMD:R_0603_1608Metric_Pad0.98x0.95mm_HandSolder
- R23: value 13.3K -> 10K; footprint Resistor_SMD:R_0805_2012Metric -> Resistor_SMD:R_0603_1608Metric_Pad0.98x0.95mm_HandSolder
- R24: value 47K -> 24K; footprint Resistor_SMD:R_0805_2012Metric -> Resistor_SMD:R_0603_1608Metric_Pad0.98x0.95mm_HandSolder
- R25: value 47K -> 100R; footprint Resistor_SMD:R_0805_2012Metric -> Resistor_SMD:R_0603_1608Metric_Pad0.98x0.95mm_HandSolder
- R27: value 100K -> 4K7; footprint Resistor_SMD:R_0805_2012Metric -> Resistor_SMD:R_0603_1608Metric_Pad0.98x0.95mm_HandSolder
- R28: value 1K -> 4K7; footprint Resistor_SMD:R_0805_2012Metric -> Resistor_SMD:R_0603_1608Metric_Pad0.98x0.95mm_HandSolder
- R29: value 1K -> 100R; footprint Resistor_SMD:R_0805_2012Metric -> Resistor_SMD:R_0603_1608Metric_Pad0.98x0.95mm_HandSolder
- R30: value 470 -> 100K; footprint Resistor_SMD:R_0805_2012Metric -> Resistor_SMD:R_0603_1608Metric_Pad0.98x0.95mm_HandSolder
- R31: value 470 -> 10K; footprint Resistor_SMD:R_0805_2012Metric -> Resistor_SMD:R_0603_1608Metric_Pad0.98x0.95mm_HandSolder
- R32, R33: value 100 -> 10K; footprint Resistor_SMD:R_0805_2012Metric -> Resistor_SMD:R_0603_1608Metric_Pad0.98x0.95mm_HandSolder
- R34: value 20K -> 100R; footprint Resistor_SMD:R_0805_2012Metric -> Resistor_SMD:R_0603_1608Metric_Pad0.98x0.95mm_HandSolder
- R35: value 20K -> 100K; footprint Resistor_SMD:R_0805_2012Metric -> Resistor_SMD:R_0603_1608Metric_Pad0.98x0.95mm_HandSolder
- R36: value 42K -> 17.6K; footprint Resistor_SMD:R_0805_2012Metric -> Resistor_SMD:R_0603_1608Metric_Pad0.98x0.95mm_HandSolder
- R37: value 35 -> 10K; footprint Resistor_SMD:R_0805_2012Metric -> Resistor_SMD:R_0603_1608Metric_Pad0.98x0.95mm_HandSolder
- R5: renamed from R19; footprint Resistor_SMD:R_0805_2012Metric -> Resistor_SMD:R_0603_1608Metric_Pad0.98x0.95mm_HandSolder
- R6: renamed from R20; footprint Resistor_SMD:R_0805_2012Metric -> Resistor_SMD:R_0603_1608Metric_Pad0.98x0.95mm_HandSolder
- R7: value 10K -> 100K; footprint Resistor_SMD:R_0805_2012Metric -> Resistor_SMD:R_0603_1608Metric_Pad0.98x0.95mm_HandSolder
- R8: value 1K -> 47K; footprint Resistor_SMD:R_0805_2012Metric -> Resistor_SMD:R_0603_1608Metric_Pad0.98x0.95mm_HandSolder
- R9: value 1K -> 45K 1%; footprint Resistor_SMD:R_0805_2012Metric -> Resistor_SMD:R_0603_1608Metric_Pad0.98x0.95mm_HandSolder
- U2: value TPS54202DDCT -> TPS2553DBVR; footprint Extra:SOT95P280X110-6N -> Extra:SOT95P280X145-6N
- U4: value TLV1117LV-3.3 -> TPS2116DRL; footprint Package_SON:WSON-8-1EP_4x4mm_P0.8mm_EP2.2x3mm -> Package_TO_SOT_SMD:SOT-583-8
- moved Q7 110.4 mm to (159.3, 109.8)
- moved Q5 109.7 mm to (159.3, 105.0)
- moved C15 106.1 mm to (188.8, 120.2)
- moved C17 104.0 mm to (181.5, 112.2), turned to -90 degrees
- moved C12 98.2 mm to (170.5, 88.6), turned to -90 degrees
- moved C10 97.9 mm to (172.6, 88.6), turned to -90 degrees
- moved C16 97.7 mm to (186.7, 105.5), turned to 90 degrees
- moved C9 96.8 mm to (174.7, 88.6), turned to -90 degrees
- moved C11 96.6 mm to (169.1, 62.4), turned to 90 degrees
- moved C13 91.4 mm to (175.2, 55.4), turned to 90 degrees
- moved C19 91.3 mm to (186.4, 100.2)
- moved L3 91.2 mm to (184.2, 103.0), turned to 90 degrees
- moved L2 91.0 mm to (184.1, 88.9), turned to 90 degrees
- moved J2 88.5 mm to (190.9, 126.5)
- moved CR1 88.2 mm to (185.1, 130.2), turned to -90 degrees
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- renumbered J5 to J1, U8 to U3, U1 to U5, U7 to U6
Connections:
- C11 pad 1: +3.3V -> Net-(U6-VPP)
- C12 pad 1: +3.3V -> +5V
- C14 pad 1: /EN -> +3.3V
- C15 pad 1: +5V -> +36V
- C16 pad 1: Net-(U7-VPP) -> Net-(U7-SS)
- C17 pad 1: +5V -> Net-(U7-SW)
- C17 pad 2: GND -> Net-(U7-BOOT)
- C18 pad 1: +3.3VA -> +3.3V
- C19 pad 1: +3.3VA -> /Vout
- C20 pad 1: +12V -> /Vout
- C21 pad 1: Net-(U2-BOOT) -> /SW
- C21 pad 2: Net-(U2-SW) -> GND
- C7 pad 1: +5V -> +3.3V
- C9 pad 1: /SW -> +5V
- CR1 pad 1: /ARM1 -> Net-(CR1-Pad1)
- CR1 pad 2: Net-(CR1-Pad2) -> GND
- D4 pad 1: Net-(D4-K) -> +36V
- F2 pad 1: Net-(D3-PadK) -> Net-(CR1-Pad1)
- F2 pad 2: Net-(U6-IN) -> +36V
- J1 pad A5: Net-(J5-CC1) -> Net-(J1-CC1)
- J1 pad B5: Net-(J5-CC2) -> Net-(J1-CC2)
- J1 pad B6: unconnected-(J5-D+-PadB6) -> /D+
- J1 pad B7: unconnected-(J5-D--PadB7) -> /D-
- J2 pad 1: GND -> Net-(CR1-Pad1)
- J2 pad 2: +3.3V -> GND
- J2 pad 3: /SDA -> (no net)
- J4 pad 1: Net-(D4-A) -> /LEFT_HAND
- J4 pad 2: GND -> /LEFT_HAND
- L1 pad 1: Net-(U2-SW) -> Net-(U4-VIN2)
- L1 pad 2: /Vout -> Net-(U2-OUT)
- L2 pad 2: Net-(U5-MODE) -> Net-(U4-MODE)
- L3 pad 1: Net-(U5-VIN2) -> Net-(U7-SW)
- L3 pad 2: Net-(U6-OUT) -> /Vout
- Q3 pad 1: Net-(Q3-G) -> Net-(Q2-Pad3)
- Q3 pad 2: /Digi_GND -> Net-(Q2-Pad1)
- Q3 pad 3: /ARM1 -> /Digi_GND
- Q4 pad 1: Net-(CR1-Pad2) -> Net-(Q4-D)
- Q4 pad 2: /ARM1 -> Net-(Q4-G)
- Q4 pad 3: +12V -> /Digi_GND
- Q5 pad 1: Net-(Q5-Pad1) -> /LEFT_HAND
- Q5 pad 2: /ARM2 -> Net-(D4-A)
- Q5 pad 3: +12V -> +36V
- Q6 pad 1: Net-(Q6-G) -> /LEFT_HAND
- Q6 pad 2: /Digi_GND -> Net-(Q6-G)
- Q6 pad 3: /ARM2 -> /Digi_GND
- Q7 pad 1: Net-(Q7-B) -> /RIGHT_HAND
- Q7 pad 2: /Digi_GND -> Net-(D5-A)
- Q7 pad 3: Net-(Q7-C) -> +36V
- Q8 pad 1: Net-(Q8-B) -> /RIGHT_HAND
- Q8 pad 2: /Digi_GND -> Net-(Q8-G)
- Q8 pad 3: Net-(Q8-C) -> /Digi_GND
- Q9 pad 1: Net-(Q10-B) -> Net-(Q9-D)
- Q9 pad 2: Net-(Q10-C) -> Net-(Q9-G)
- R10 pad 1: /LED_B -> Net-(U4-MODE)
- R10 pad 2: Net-(D1-BK) -> Net-(U4-PR1)
- R11 pad 1: +3.3V -> Net-(U4-PR1)
- R11 pad 2: /SCL -> GND
- R12 pad 2: /SDA -> /EN
- R13 pad 1: Net-(U6-IN) -> +3.3V
- R13 pad 2: Net-(U6-EN) -> /power_mux
- R14 pad 2: /EN -> Net-(U6-~{RST})
- R21 pad 1: /Vout -> /GPIO17
- R21 pad 2: Net-(C24-Pad1) -> /Digi_GND
- R22 pad 1: Net-(C24-Pad1) -> +36V
- R22 pad 2: Net-(R22-Pad2) -> Net-(D4-A)
- R23 pad 1: Net-(R22-Pad2) -> Net-(D4-A)
- R23 pad 2: GND -> Net-(Q4-D)
- R24 pad 1: +12V -> Net-(U7-RT_SYNC)
- R24 pad 2: Net-(Q7-C) -> GND
- R25 pad 1: +12V -> /GPIO17
- R25 pad 2: Net-(Q8-C) -> Net-(Q6-G)
- R26 pad 1: /GPIO17 -> +36V
- R26 pad 2: /Digi_GND -> Net-(U7-EN)
- R27 pad 1: /GPIO16 -> +3.3V
- R27 pad 2: /Digi_GND -> /SDA
- R28 pad 1: Net-(Q7-B) -> +3.3V
- R28 pad 2: /GPIO16 -> /SCL
- R29 pad 1: Net-(Q8-B) -> Net-(Q8-G)
- R29 pad 2: /GPIO17 -> /GPIO16
- R30 pad 1: Net-(CR1-Pad2) -> +36V
- R30 pad 2: Net-(Q7-C) -> Net-(D5-A)
- R31 pad 1: Net-(Q8-C) -> Net-(D5-A)
- R31 pad 2: Net-(Q5-Pad1) -> Net-(Q9-D)
- R32 pad 1: Net-(Q3-G) -> /GPIO16
- R32 pad 2: /GPIO17 -> /Digi_GND
- R33 pad 1: /GPIO16 -> +3.3V
- R33 pad 2: Net-(Q6-G) -> /SW
- R34 pad 1: Net-(CR1-Pad2) -> Net-(Q9-G)
- R34 pad 2: /ARM1 -> /GPIO17
- R35 pad 1: Net-(Q5-Pad1) -> /Vout
- R35 pad 2: /ARM2 -> Net-(U7-FB)
- R36 pad 1: +12V -> Net-(U7-FB)
- R36 pad 2: Net-(Q10-C) -> GND
- R37 pad 1: Net-(Q10-B) -> /GPIO17
- R37 pad 2: GND -> /Digi_GND
- R5 pad 1: GND -> Net-(J1-CC2)
- R5 pad 2: Net-(J5-CC1) -> GND
- R6 pad 1: GND -> Net-(J1-CC1)
- R6 pad 2: Net-(J5-CC2) -> GND
- R7 pad 1: +3.3V -> Net-(U2-IN)
- R7 pad 2: /SW -> Net-(U2-EN)
- R8 pad 1: /LED_R -> +3.3V
- R8 pad 2: Net-(D1-RK) -> /FAULT
- R9 pad 1: /LED_G -> Net-(U2-ILIM)
- R9 pad 2: Net-(D1-GK) -> GND
- U2 pad 1: GND -> Net-(U2-IN)
- U2 pad 2: Net-(U2-SW) -> GND
- U2 pad 3: +12V -> Net-(U2-EN)
- U2 pad 4: GND -> /FAULT
- U2 pad 5: unconnected-(U2-EN-Pad5) -> Net-(U2-ILIM)
- U2 pad 6: Net-(U2-BOOT) -> Net-(U2-OUT)
- U4 pad 1: unconnected-(U4-GND-Pad1) -> GND
- U4 pad 3: +5V -> Net-(U4-MODE)
- U4 pad 4: +5V -> Net-(U4-PR1)
- U4 pad 5: +3.3V -> Net-(U4-MODE)
- U4 pad 6: +3.3V -> Net-(U4-VIN2)
- U4 pad 7: +3.3V -> +5V
- U4 pad 8: unconnected-(U4-NC-Pad8) -> /power_mux
- U5 pad 34: /TX -> /RX
- U5 pad 35: /RX -> /TX
- U5 pad 6: /GPIO34 -> /power_mux
- U6 pad 16: Net-(U7-VPP) -> Net-(U6-VPP)
- U6 pad 5: +3.3VA -> +3.3V
- U6 pad 6: +3.3VA -> +3.3V
- U6 pad 9: Net-(U7-~{RST}) -> Net-(U6-~{RST})
Routing:
- net +3.3V: track 0.00 -> 70.4 mm, vias 0 -> 2
- net +5V: track 0.00 -> 58.3 mm, vias 0 -> 3
- net GND: track 0.00 -> 47.3 mm, vias 0 -> 27
- net Net-(U4-MODE): track 0.00 -> 27.1 mm
- net Net-(U7-FB): track 0.00 -> 22.9 mm
- net /TX: track 30.4 -> 11.2 mm, vias 2 -> 0
- net /RX: track 27.9 -> 8.82 mm, vias 2 -> 0
- net /Vout: track 0.00 -> 18.0 mm
- net +5VP: track 0.00 -> 14.4 mm
- net Net-(U2-IN): track 0.00 -> 12.4 mm
- net +36V: track 0.00 -> 11.9 mm
- net Net-(CR1-Pad1): track 0.00 -> 10.5 mm
- net Net-(U4-VIN2): track 0.00 -> 9.88 mm
- net Net-(U7-SW): track 0.00 -> 9.37 mm
- net Net-(U4-PR1): track 0.00 -> 9.36 mm
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
Commit message: First Complete Draft done
Parts:
- removed Q8, Q9: AON6266E, Extra:AON6482
- added MOSFET1: FDC5614P, Extra:TSOT23-6_419BL_ONS, F.Cu at (172.0, 115.1)
- added MOSFET2: FDC5614P, Extra:TSOT23-6_419BL_ONS, F.Cu at (172.0, 124.5)
- Q4, Q6: value AON6266E -> T2N7002BK_LM; footprint Extra:AON6482 -> Extra:SOT23_TOS-M
- Q5, Q7: value FDC5614P -> T2N7002BK_LM; footprint Extra:TSOT23-6_419BL_ONS -> Extra:SOT23_TOS-M
- moved SW1 134.1 mm to (131.0, 85.9)
- moved J3 116.7 mm to (128.3, 97.1)
- moved Q1 114.1 mm to (144.9, 97.8)
- moved R12 109.8 mm to (130.5, 54.6)
- moved Q2 109.1 mm to (150.7, 105.8)
- moved R19 105.0 mm to (136.2, 82.2), turned to -90 degrees
- moved C7 92.5 mm to (136.0, 53.5), turned to -90 degrees
- moved R18 91.5 mm to (144.5, 106.8), turned to 180 degrees
- moved C8 89.1 mm to (137.7, 53.5), turned to -90 degrees
- moved R37 86.8 mm to (160.0, 127.3), turned to 180 degrees
- moved R34 86.2 mm to (164.8, 131.0)
- moved C4 85.6 mm to (138.0, 57.7), turned to 180 degrees
- moved R15 85.0 mm to (150.5, 97.9), turned to 180 degrees
- moved Q6 84.9 mm to (162.6, 122.5), turned to 90 degrees
- moved R33 84.5 mm to (162.8, 119.2), turned to 180 degrees
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- renumbered C21 to C15, C15 to C16, C16 to C17, C17 to C18, C18 to C19, C19 to C20, C20 to C21, Q2 to Q1, Q3 to Q2, Q1 to Q3, R17 to R15, R15 to R16, R16 to R17, R19 to R18, R33 to R19, R18 to R20, R20 to R21, R21 to R24, R24 to R25, R25 to R26, R26 to R27, R27 to R28, R28 to R29, R29 to R30, R30 to R31, R31 to R32, R32 to R33
Connections:
- C11 pad 2: GND -> +3.3V
- J3 pad 10: /GPIO27 -> GND
- J3 pad 4: /GPIO18 -> /GPIO27
- J3 pad 6: /GPIO25 -> /GPIO19
- J3 pad 7: /GPIO34 -> /GPIO25
- J3 pad 8: /GPIO26 -> /GPIO18
- J3 pad 9: GND -> /GPIO26
- Q5 pad 2: Net-(D4-A) -> Net-(Q5-G)
- Q5 pad 3: +36V -> /Digi_GND
- Q6 pad 1: /LEFT_HAND -> /RIGHT_HAND
- Q7 pad 1: /RIGHT_HAND -> Net-(Q7-D)
- Q7 pad 2: Net-(D5-A) -> Net-(Q7-G)
- Q7 pad 3: +36V -> /Digi_GND
- R26 pad 2: Net-(Q6-G) -> Net-(Q5-G)
- R30 pad 1: Net-(Q8-G) -> Net-(Q6-G)
- R32 pad 2: Net-(Q9-D) -> Net-(Q7-D)
- R34 pad 1: Net-(Q9-G) -> Net-(Q7-G)
- U7 pad V: (no net) -> GND
Routing:
- net +36V: track 11.9 -> 122.4 mm
- net /GPIO17: track 0.00 -> 88.1 mm, vias 0 -> 3
- net +3.3V: track 70.4 -> 157.1 mm, vias 2 -> 8
- net /EN: track 0.00 -> 80.0 mm, vias 0 -> 2
- net GND: track 47.3 -> 125.7 mm, vias 27 -> 42
- net /GPIO16: track 0.00 -> 77.0 mm, vias 0 -> 3
- net /power_mux: track 2.19 -> 74.6 mm, vias 0 -> 2
- net /Digi_GND: track 0.00 -> 71.4 mm
- net /GPIO26: track 0.00 -> 67.5 mm, vias 0 -> 2
- net /FAULT: track 0.00 -> 67.1 mm, vias 0 -> 4
- net /GPIO25: track 0.00 -> 64.6 mm, vias 0 -> 2
- net /GPIO33: track 0.00 -> 62.2 mm, vias 0 -> 2
- net /SW: track 0.00 -> 61.4 mm, vias 0 -> 2
- net /GPIO19: track 0.00 -> 59.8 mm, vias 0 -> 2
- net /GPIO32: track 0.00 -> 59.4 mm, vias 0 -> 2
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- added copper zone on In2.Cu, net +3.3V
- added copper zone on In2.Cu, net +5V
- added copper zone on F.Cu, net /LEFT_HAND
- added copper zone on F.Cu, net /RIGHT_HAND
- added copper zone on In1.Cu, net GND
Other:
- board size 100 x 100 mm -> 81 x 99.9 mm

Commit message: Finished PCB
Parts:
- moved R6 2.94 mm to (186.6, 65.1)
- moved R5 2.81 mm to (186.6, 61.3)
- moved D1 0.80 mm to (188.3, 67.9)
- moved F1 0.80 mm to (186.4, 67.8)
- moved J1 0.46 mm to (197.1, 63.2)
- moved H3 0.28 mm to (121.7, 141.3)
- moved H2 0.28 mm to (195.3, 48.8)
- moved H4 0.28 mm to (195.3, 141.3)
- moved H1 0.14 mm to (121.7, 48.8)
Routing:
- net /D+: track 11.6 -> 26.4 mm, vias 0 -> 2
- net /D-: track 11.6 -> 26.4 mm, vias 0 -> 2
- net Net-(D4-A): track 7.75 -> 16.4 mm, vias 0 -> 2
- net /RIGHT_HAND: track 38.4 -> 45.4 mm
- net /LEFT_HAND: track 56.7 -> 63.1 mm
- net Net-(J1-CC1): track 2.30 -> 4.81 mm
- net Net-(J1-CC2): track 2.18 -> 4.55 mm
- net +3.3V: track 157.1 -> 158.9 mm

Commit message: meow
Parts:
- added Pot1: 1, Resistor_THT:R_Axial_DIN0204_L3.6mm_D1.6mm_P2.54mm_Vertical, F.Cu at (138.3, 126.5)
- added R38: 5000, Resistor_SMD:R_0603_1608Metric_Pad0.98x0.95mm_HandSolder, F.Cu at (139.1, 122.0)
Connections:
- U7 pad V: GND -> (no net)
Routing:
- net +3.3V: track 158.9 -> 203.3 mm, vias 8 -> 9
- net unconnected-(Pot1-Pad1): track 0.00 -> 4.54 mm
- net GND: track 125.9 -> 127.9 mm

Commit message: Update
Parts:
- removed Pot1: 1, Resistor_THT:R_Axial_DIN0204_L3.6mm_D1.6mm_P2.54mm_Vertical
- added J7: PDB181-K420K-502B, Extra:CONN3_PDB181-K420K-502B_BRN, F.Cu at (154.8, 141.4)
- added R39: PTV09A-4015U-A204, Extra:POT_PTV09A-4x15x-xxxx_BRN, F.Cu at (135.6, 126.4)
- added R40: 0R, Resistor_SMD:R_0603_1608Metric_Pad0.98x0.95mm_HandSolder, F.Cu at (149.4, 133.4)
- moved R38 2.96 mm to (142.0, 122.5)
- moved R25 1.03 mm to (190.8, 116.2)
- moved C15 0.65 mm to (165.1, 53.6)
- moved R26 0.42 mm to (166.9, 110.9)
- moved U5 0.12 mm to (150.0, 61.1)
Connections:
- MOSFET2 pad 1: /RIGHT_HAND -> Net-(Q6-D)
- MOSFET2 pad 2: /RIGHT_HAND -> Net-(Q6-D)
- MOSFET2 pad 5: /RIGHT_HAND -> Net-(Q6-D)
- MOSFET2 pad 6: /RIGHT_HAND -> Net-(Q6-D)
- Q6 pad 1: /RIGHT_HAND -> Net-(Q6-D)
Routing:
- net unconnected-(R38-Pad2): track 4.54 -> 72.7 mm, vias 0 -> 2
- net Net-(Q6-D): track 0.00 -> 42.3 mm, vias 0 -> 3
- net GND: track 127.9 -> 163.5 mm, vias 42 -> 45
- net /RIGHT_HAND: track 45.4 -> 29.5 mm, vias 2 -> 0
- net /Digi_GND: track 71.4 -> 82.1 mm, vias 0 -> 3
- net +36V: track 122.4 -> 128.5 mm, vias 0 -> 3
- net /Vout: track 18.0 -> 23.5 mm, vias 0 -> 2
- net /power_mux: track 74.6 -> 79.9 mm, vias 2 -> 3
- net +5VP: track 14.0 -> 19.1 mm, vias 0 -> 1
- net +5V: track 58.3 -> 62.0 mm, vias 3 -> 5
- net +3.3V: track 203.3 -> 207.0 mm, vias 9 -> 11
- net /LEFT_HAND: track 63.1 -> 66.1 mm, vias 2 -> 3
- net Net-(D5-A): track 17.1 -> 20.1 mm, vias 0 -> 2
- net Net-(U6-TXD): track 11.7 -> 13.7 mm, vias 0 -> 1
- net Net-(D4-A): track 16.4 -> 18.2 mm, vias 2 -> 3
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- added copper zone on F.Cu, net Net-(Q6-D)
- removed copper zone on F.Cu, net /RIGHT_HAND
Other:
- board text added: "D & D"
- board text added: "T1"
- board text added: "T10"
- board text added: "T11"
- board text added: "T12"
- board text added: "T13"
- board text added: "T14"
- board text added: "T15"
- board text added: "T16"
- board text added: "T17"
- board text added: "T18"
- board text added: "T19"
- board text added: "T2"
- board text added: "T20"
- board text added: "T21"
- board text added: "T22"
- board text added: "T23"
- board text added: "T24"
- board text added: "T25"
- board text added: "T26"
- board text added: "T27"
- board text added: "T28"
- board text added: "T29"
- board text added: "T3"
- board text added: "T30A"
- board text added: "T31A"
- board text added: "T31B"
- board text added: "T4"
- board text added: "T5"
- board text added: "T6"
- board text added: "T7"
- board text added: "T8"
- board text added: "T9"
